Commit message: New basic sr300 model. Improved pick and draw.

File: turtlebot/turtlebot_description/urdf/sensors/sr300.urdf.xacro (robot description, xacro)
@@ -4,5 +4,5 @@
   <xacro:include filename="$(find turtlebot_description)/urdf/turtlebot_properties.urdf.xacro"/>
   <!-- Intel SR300 parameters -->
-  <xacro:property name="sr300_cam_offset_px" value="0.140" />
+  <xacro:property name="sr300_cam_offset_px" value="0.142" />
   <xacro:property name="sr300_cam_offset_py" value="0.0" />
   <xacro:property name="sr300_cam_offset_pz" value="0.39" />
@@ -29,5 +29,5 @@
     <link name="camera_sr300">
       <visual>
-       <origin xyz="0 0 0" rpy="${M_PI/2} 0 ${M_PI/2}"/>
+       <origin xyz="0 0 0" rpy="0 0 0"/>
         <geometry>
          <mesh filename="package://turtlebot_description/meshes/sensors/sr300.stl" />
@@ -36,5 +36,5 @@
       </visual>
       <collision>
-        <origin xyz="0.0 0.0 0.0" rpy="${M_PI/2} 0 ${M_PI/2}"/>
+        <origin xyz="0.0 0.0 0.0" rpy="0 0 0"/>
         <geometry>
           <mesh filename="package://turtlebot_description/meshes/sensors/sr300.stl" scale="2.0 2.0 2.0" />
