Commit message: Positioned MK3 arm with new mount

File: turtlebot/turtlebot_description/robots/kobuki_interbotix_astra.urdf.xacro (robot description, xacro)
@@ -11,7 +11,7 @@
   <stack_interbotix parent="base_link"/>
   <sensor_astra parent="base_link"/>
-  <sensor_sr300  parent="base_link"/>
+  <sensor_sr300 parent="base_link"/>
   <phantomx_pincher_arm parent="base_link" color="Red" gripper_color="Red">
-    <origin xyz="0.135 0.0 0.1125"/>
+    <origin xyz="0.142 0.0 0.112"/>
   </phantomx_pincher_arm>
 </robot>

File: turtlebot/turtlebot_description/robots/kobuki_interbotix_zr300.urdf.xacro (robot description, xacro)
@@ -13,5 +13,5 @@
   <sensor_sr300 parent="base_link"/>
   <phantomx_pincher_arm parent="base_link" color="Red" gripper_color="Red">
-    <origin xyz="0.135 0.0 0.1125"/>
+    <origin xyz="0.142 0.0 0.112"/>
   </phantomx_pincher_arm>
 </robot>
