Commit message: Initial Pincher MK3 Description

File: phantomx_pincher_arm/phantomx_pincher_arm_description/urdf/phantomx_pincher_gripper.xacro (robot description, xacro)
@@ -1,43 +1,35 @@
 <?xml version="1.0"?>
-<!-- PhantomX Pincher Arm gripper URDF-->
+<!-- PhantomX Pincher gripper URDF-->
 <robot xmlns:xacro="http://ros.org/wiki/xacro">
-    <bioloid_F3_fixed parent="arm_wrist_flex_link" name="arm_wrist_F3_0" color="${color}">
-      <origin xyz="0 0 ${F2_HEIGHT}" rpy="0 ${M_PI} ${-M_PI}"/>
-    </bioloid_F3_fixed>
     <!-- gripper joint -->
-    <dynamixel_AX12_fixed parent="arm_wrist_F3_0_link" name="gripper_servo" >
-      <origin xyz="0 0 ${-AX12_WIDTH/2}" rpy="${M_PI/2} ${M_PI} ${M_PI/2}"/>
-    </dynamixel_AX12_fixed>
-     <gripper_finger_base parent="gripper_servo_link" name="gripper_finger_base" color="${color}">
-      <origin xyz="0.016  ${AX12_WIDTH} 0" rpy="${M_PI/2} ${-M_PI} ${M_PI/2}"/>
-    </gripper_finger_base>
-     <!-- Finger 1 -->
+    <!-- Finger 1 -->
     <joint name="gripper_joint" type="prismatic">
-      <origin xyz="0 0 0" rpy="0 0 0"/>
-      <axis xyz="1 0 0"/>
-      <limit effort="30" velocity="0.5" lower="0.002" upper="0.031"/>
-      <parent link="gripper_servo_link"/>
+      <origin xyz="0.070 0 0" rpy="0 0 0"/>
+      <axis xyz="0 1 0"/>
+      <limit effort="30" velocity="0.5" lower="0.002" upper="0.016"/>
+      <parent link="arm_wrist_flex_link"/>
       <child link="gripper_active_link"/>
     </joint>
-    <phantomx_pincher_gripper name="gripper_active" color="${color}" >
-      <origin xyz="-0.015 0.023 0" rpy="${-M_PI/2} 0 0"/>
-    </phantomx_pincher_gripper>
+    <pincher_finger name="gripper_active" color="${color}" >
+      <origin xyz="0 0 0" rpy="0 0 0"/>
+    </pincher_finger>
     <!-- Finger 2 -->
     <!-- Note: currently static but should be a Mimic of Finger 1 -->
     <joint name="gripper2_joint" type="fixed">
-      <parent link="gripper_servo_link"/>
+      <origin xyz="0.070 -0.016 0" rpy="0 0 0"/>
+      <parent link="arm_wrist_flex_link"/>
       <child link="gripper_active2_link"/>
     </joint>
-    <phantomx_pincher_gripper name="gripper_active2" color="${color}" >
-      <origin xyz="-0.015 0.023 0" rpy="${-M_PI/2} ${M_PI} 0"/>
-    </phantomx_pincher_gripper>
+    <pincher_finger name="gripper_active2" color="${color}" >
+      <origin xyz="0 0 0" rpy="${M_PI} 0 0"/>
+    </pincher_finger>
     <!-- Using Mimic -->
     <!-- gripper 2 joint -->
-    <!--  ### Mimic would be better but causes some error
-      <joint name="gripper2_joint" type="prismatic">
-      <origin xyz="0 0 0" rpy="0 0 0"/>
-      <axis xyz="1 0 0"/>
-      <limit effort="30" velocity="0.5" lower="-0.031" upper="-0.002"/>
-      <parent link="gripper_servo_link"/>
+    <!--  TODO: Test Mimic ->
+    <joint name="gripper2_joint" type="prismatic">
+      <origin xyz="0.070 0 0" rpy="0 0 0"/>
+      <axis xyz="0 1 0"/>
+      <limit effort="30" velocity="0.5" lower="-0.016" upper="-0.002"/>
+      <parent link="arm_wrist_flex_link"/>
       <child link="gripper_active2_link"/>
       <mimic joint="gripper_joint" multiplier="-1"  offset = "0"/>
