Commit message: Fixed origin and gripper upper limit.

File: phantomx_pincher_arm/phantomx_pincher_arm_description/urdf/phantomx_pincher_arm.xacro (robot description, xacro)
@@ -7,5 +7,5 @@
     <!-- arm base link -->
     <pincher_base parent="${parent}" name="arm_base">
-      <origin xyz="0 0 0.020" rpy="0 0 0"/>
+      <xacro:insert_block name="origin"/>
     </pincher_base>
     <bracket_F2_revolute parent="arm_base_link" name="arm_shoulder_pan" color="${color}"

File: phantomx_pincher_arm/phantomx_pincher_arm_description/urdf/phantomx_pincher_gripper.xacro (robot description, xacro)
@@ -7,5 +7,5 @@
       <origin xyz="0.070 0 0" rpy="0 0 0"/>
       <axis xyz="0 1 0"/>
-      <limit effort="30" velocity="0.5" lower="0.002" upper="0.016"/>
+      <limit effort="30" velocity="0.5" lower="0.002" upper="0.032"/>
       <parent link="arm_wrist_flex_link"/>
       <child link="gripper_active_link"/>
