Commit message: Updated joint limits for MK3

File: phantomx_pincher_arm/phantomx_pincher_arm_description/urdf/phantomx_pincher_arm.urdf.xacro (robot description, xacro)
@@ -5,12 +5,12 @@
     to allow access to different operational areas, e.g. left handed vs. right handed robot -->
     <xacro:property name="joints_vlimit" value="1.571"/>
-    <xacro:property name="pan_llimit" value="-2.617"/>
-    <xacro:property name="pan_ulimit" value="2.617"/>
-    <xacro:property name="shoulder_llimit" value="-2.3"/>
-    <xacro:property name="shoulder_ulimit" value="2.3"/>
-    <xacro:property name="elbow_llimit" value="-2.42"/>
-    <xacro:property name="elbow_ulimit" value="2.38"/>
-    <xacro:property name="wrist_llimit" value="-1.72"/>
-    <xacro:property name="wrist_ulimit" value="1.68"/>
+    <xacro:property name="pan_llimit" value="-1.74"/>
+    <xacro:property name="pan_ulimit" value="1.74"/>
+    <xacro:property name="shoulder_llimit" value="-1.98"/>
+    <xacro:property name="shoulder_ulimit" value="1.88"/>
+    <xacro:property name="elbow_llimit" value="-1.58"/>
+    <xacro:property name="elbow_ulimit" value="0.59"/>
+    <xacro:property name="wrist_llimit" value="-1.79"/>
+    <xacro:property name="wrist_ulimit" value="1.67"/>
     <!-- Included URDF Files -->
     <xacro:include filename="$(find phantomx_pincher_arm_description)/urdf/phantomx_pincher_arm.xacro"/>

File: turtlebot/turtlebot_description/robots/kobuki_interbotix_astra.urdf.xacro (robot description, xacro)
@@ -13,5 +13,5 @@
   <sensor_sr300 parent="base_link"/>
   <phantomx_pincher_arm parent="base_link" color="Red" gripper_color="Red">
-    <origin xyz="0.142 0.0 0.112"/>
+    <origin xyz="0.145 0.0 0.112"/>
   </phantomx_pincher_arm>
 </robot>

File: turtlebot/turtlebot_description/robots/kobuki_interbotix_zr300.urdf.xacro (robot description, xacro)
@@ -13,5 +13,5 @@
   <sensor_sr300 parent="base_link"/>
   <phantomx_pincher_arm parent="base_link" color="Red" gripper_color="Red">
-    <origin xyz="0.142 0.0 0.112"/>
+    <origin xyz="0.145 0.0 0.112"/>
   </phantomx_pincher_arm>
 </robot>

File: turtlebot/turtlebot_description/urdf/arms/phantomx_pincher_arm.urdf.xacro (robot description, xacro)
@@ -5,12 +5,12 @@
           to allow access to different operational areas, e.g. left handed vs. right handed robot -->
     <xacro:property name="joints_vlimit" value="1.571"/>
-    <xacro:property name="pan_llimit" value="-2.617"/>
-    <xacro:property name="pan_ulimit" value="2.617"/>
-    <xacro:property name="shoulder_llimit" value="-2.617"/>
-    <xacro:property name="shoulder_ulimit" value="2.617"/>
-    <xacro:property name="elbow_llimit" value="-2.42"/>
-    <xacro:property name="elbow_ulimit" value="2.38"/>
-    <xacro:property name="wrist_llimit" value="-1.72"/>
-    <xacro:property name="wrist_ulimit" value="1.68"/>
+    <xacro:property name="pan_llimit" value="-1.74"/>
+    <xacro:property name="pan_ulimit" value="1.74"/>
+    <xacro:property name="shoulder_llimit" value="-1.98"/>
+    <xacro:property name="shoulder_ulimit" value="1.88"/>
+    <xacro:property name="elbow_llimit" value="-1.58"/>
+    <xacro:property name="elbow_ulimit" value="0.59"/>
+    <xacro:property name="wrist_llimit" value="-1.79"/>
+    <xacro:property name="wrist_ulimit" value="1.67"/>
     <!-- Included URDF Files -->
     <xacro:include filename="$(find phantomx_pincher_arm_description)/urdf/phantomx_pincher_arm.xacro" />

File: turtlebot/turtlebot_description/urdf/sensors/sr300.urdf.xacro (robot description, xacro)
@@ -6,5 +6,5 @@
   <xacro:property name="sr300_cam_offset_px" value="0.142" />
   <xacro:property name="sr300_cam_offset_py" value="0.0" />
-  <xacro:property name="sr300_cam_offset_pz" value="0.39" />
+  <xacro:property name="sr300_cam_offset_pz" value="0.428" />
   <!--
   <xacro:property name="sr300_cam_rgb_px" value="0.005"/>

File: turtlebot/turtlebot_description/urdf/sensors/zr300.urdf.xacro (robot description, xacro)
@@ -6,5 +6,5 @@
   <xacro:property name="zr300_origin_x" value="-0.050"/>
   <xacro:property name="zr300_origin_y" value="0.0"/>
-  <xacro:property name="zr300_origin_z" value="0.230"/>
+  <xacro:property name="zr300_origin_z" value="0.268"/>
   <xacro:property name="zr300_rgb_x" value="0.0"/>
   <xacro:property name="zr300_rgb_y" value="-0.028"/>

File: turtlebot/turtlebot_description/urdf/stacks/interbotix.urdf.xacro (robot description, xacro)
@@ -220,5 +220,5 @@
         <origin xyz="0.0 0.0 0.0" rpy="0 0 0"/>
         <geometry>
-          <mesh filename="package://turtlebot_description/meshes/stacks/interbotix/plate_middle.stl"/>
+          <mesh filename="package://turtlebot_description/meshes/stacks/interbotix/plate_middle.stl" scale="1.1 1.1 1.1"/>
         </geometry>
       </collision>
@@ -313,5 +313,5 @@
     <standoff_38mm parent="${parent}" number="13" x_loc="-0.104" y_loc="-0.098" z_loc="0.378"/>
     <joint name="plate_top_joint" type="fixed">
-      <origin xyz="0.0 0.0 0.3995" rpy="0 0 0"/>
+      <origin xyz="0.0 0.0 0.4375" rpy="0 0 0"/>
       <parent link="${parent}"/>
       <child link="plate_top_link"/>
