Commit message: Moving plates to new positions

File: turtlebot/turtlebot_description/urdf/stacks/interbotix.urdf.xacro (robot description, xacro)
@@ -241,5 +241,5 @@
     <standoff_38mm parent="${parent}" number="9" x_loc="-0.104" y_loc="-0.098" z_loc="0.206"/>
     <joint name="plate_utility_lower" type="fixed">
-      <origin xyz="0.0 0.0 0.2275" rpy="0 0 0"/>
+      <origin xyz="0.0 0.0 0.2655" rpy="0 0 0"/>
       <parent link="${parent}"/>
       <child link="plate_utility_lower_link"/>

Commit message: Updated URDF and SRDF

File: turtlebot/turtlebot_description/urdf/stacks/interbotix.urdf.xacro (robot description, xacro)
@@ -1,16 +1,32 @@
 <?xml version="1.0"?>
-<!--
-  Interbotix stacks
- -->
 <robot name="stack_interbotix" xmlns:xacro="http://ros.org/wiki/xacro">
+  <!-- TODO: Intertia fields do not contain valid data. Follow tutorial to correct them: http://gazebosim.org/tutorials?tut=inertia -->
   <xacro:include filename="$(find turtlebot_description)/urdf/common_properties.urdf.xacro"/>
   <!-- Xacro properties -->
+  <xacro:property name="PLATE_HEIGHT" value="0.0046"/>
+  <xacro:property name="STANDOFF_38_HEIGHT" value="0.038"/>
+  <xacro:property name="STANDOFF_51_HEIGHT" value="0.051"/>
+  <xacro:property name="STANDOFF_81_HEIGHT" value="${STANDOFF_38_HEIGHT*2.0+PLATE_HEIGHT}"/>
+  <xacro:property name="STANDOFF_251_HEIGHT" value="${STANDOFF_38_HEIGHT*6.0+PLATE_HEIGHT*5.0}"/>
+  <xacro:property name="KOBUKI_TOP_HEIGHT" value="0.0975"/> <!--Measure the floor to the top of the robot base where the standoffs install-->
+  <xacro:property name="BASE_LINK_HEIGHT" value="0.0102"/> <!--TODO: Base link for turtlebot is 10.2mm from floor. Why? -->
+  <xacro:property name="STANDOFF_BOTTOM_Z" value="${KOBUKI_TOP_HEIGHT+STANDOFF_38_HEIGHT/2.0-BASE_LINK_HEIGHT}"/>
+  <xacro:property name="PLATE_BOTTOM_Z" value="${STANDOFF_BOTTOM_Z+STANDOFF_38_HEIGHT/2.0+PLATE_HEIGHT/2.0}"/>
+  <xacro:property name="STANDOFF_MIDDLE_Z" value="${PLATE_BOTTOM_Z+PLATE_HEIGHT/2.0+STANDOFF_51_HEIGHT/2.0}"/>
+  <xacro:property name="PLATE_MIDDLE_Z" value="${STANDOFF_MIDDLE_Z+STANDOFF_51_HEIGHT/2.0+PLATE_HEIGHT/2.0}"/>
+  <xacro:property name="STANDOFF_UTILITY_BOTTOM_Z" value="${PLATE_MIDDLE_Z+PLATE_HEIGHT/2.0+STANDOFF_81_HEIGHT/2.0}"/>
+  <xacro:property name="PLATE_UTILITY_BOTTOM_Z" value="${STANDOFF_UTILITY_BOTTOM_Z+STANDOFF_81_HEIGHT/2.0+PLATE_HEIGHT/2.0}"/>
+  <xacro:property name="STANDOFF_UTILITY_UPPER_Z" value="${PLATE_UTILITY_BOTTOM_Z+PLATE_HEIGHT/2.0+STANDOFF_81_HEIGHT/2.0}"/>
+  <xacro:property name="PLATE_UTILITY_UPPER_Z" value="${STANDOFF_UTILITY_UPPER_Z+STANDOFF_81_HEIGHT/2.0+PLATE_HEIGHT/2.0}"/>
+  <xacro:property name="STANDOFF_TOP_Z" value="${PLATE_UTILITY_UPPER_Z+PLATE_HEIGHT/2.0+STANDOFF_81_HEIGHT/2.0}"/>
+  <xacro:property name="PLATE_TOP_Z" value="${STANDOFF_TOP_Z+STANDOFF_81_HEIGHT/2.0+PLATE_HEIGHT/2.0}"/>
+  <xacro:property name="STANDOFF_FRONT_Z" value="${PLATE_MIDDLE_Z+PLATE_HEIGHT/2.0+STANDOFF_251_HEIGHT/2.0}"/>
   <xacro:property name="material_pink">
-    <material name="orange">
+    <material name="pink">
       <color rgba="0.8 0.0 0.4 1"/>
     </material>
   </xacro:property>
   <xacro:property name="material_near_black">
-    <material name="black">
+    <material name="near_black">
       <color rgba="0.125 0.125 0.125 1"/>
     </material>
@@ -28,5 +44,5 @@
         <origin xyz="0 0 0" rpy="0 0 0"/>
         <geometry>
-          <mesh filename="package://turtlebot_description/meshes/stacks/interbotix/standoff_38mm.stl"/>
+          <mesh filename="package://turtlebot_description/meshes/stacks/interbotix/38mm_HexStandoff_MF.stl"/>
         </geometry>
         <xacro:insert_block name="material_pink"/>
@@ -35,5 +51,5 @@
         <origin xyz="0 0 0" rpy="0 0 0"/>
         <geometry>
-          <cylinder length="0.038" radius="0.006"/>
+          <cylinder length="${STANDOFF_38_HEIGHT}" radius="0.006"/>
         </geometry>
       </collision>
@@ -62,5 +78,5 @@
         <origin xyz="0 0 0" rpy="0 ${M_PI} 0"/>
         <geometry>
-          <mesh filename="package://turtlebot_description/meshes/stacks/interbotix/standoff_51mm.stl"/>
+          <mesh filename="package://turtlebot_description/meshes/stacks/interbotix/51mm_HexStandoff_FF.stl"/>
         </geometry>
         <xacro:insert_block name="material_pink"/>
@@ -69,5 +85,5 @@
         <origin xyz="0 0 0" rpy="0 0 0"/>
         <geometry>
-          <cylinder length="0.051" radius="0.006"/>
+          <cylinder length="${STANDOFF_51_HEIGHT}" radius="0.006"/>
         </geometry>
       </collision>
@@ -86,15 +102,15 @@
     </gazebo>
   </xacro:macro>
-  <xacro:macro name="standoff_124mm" params="parent number x_loc y_loc z_loc">
-    <joint name="standoff_124mm_${number}_joint" type="fixed">
+  <xacro:macro name="standoff_81mm" params="parent number x_loc y_loc z_loc">
+    <joint name="standoff_81mm_${number}_joint" type="fixed">
       <origin xyz="${x_loc} ${y_loc} ${z_loc}" rpy="0 0 0"/>
       <parent link="${parent}"/>
-      <child link="standoff_124mm_${number}_link"/>
-    </joint>
-    <link name="standoff_124mm_${number}_link">
+      <child link="standoff_81mm_${number}_link"/>
+    </joint>
+    <link name="standoff_81mm_${number}_link">
       <visual>
         <origin xyz=" 0 0 0" rpy="0 0 0"/>
         <geometry>
-          <mesh filename="package://turtlebot_description/meshes/stacks/interbotix/standoff_124mm.stl"/>
+          <mesh filename="package://turtlebot_description/meshes/stacks/interbotix/81mm_Spacer.stl"/>
         </geometry>
         <xacro:insert_block name="material_pink"/>
@@ -103,5 +119,5 @@
         <origin xyz="0 0 0" rpy="0 0 0"/>
         <geometry>
-          <cylinder length="0.124" radius="0.012"/>
+          <cylinder length="${STANDOFF_81_HEIGHT}" radius="0.012"/>
         </geometry>
       </collision>
@@ -114,21 +130,21 @@
       </inertial>
     </link>
-    <gazebo reference="standoff_124mm_${number}_link">
-      <material>Gazebo/Black</material>
-      <selfCollide>true</selfCollide>
-      <gravity>true</gravity>
-    </gazebo>
-  </xacro:macro>
-  <xacro:macro name="standoff_209mm" params="parent number x_loc y_loc z_loc">
-    <joint name="standoff_209mm_${number}_joint" type="fixed">
+    <gazebo reference="standoff_81mm_${number}_link">
+      <material>Gazebo/Black</material>
+      <selfCollide>true</selfCollide>
+      <gravity>true</gravity>
+    </gazebo>
+  </xacro:macro>
+  <xacro:macro name="standoff_251mm" params="parent number x_loc y_loc z_loc">
+    <joint name="standoff_251mm_${number}_joint" type="fixed">
       <origin xyz="${x_loc} ${y_loc} ${z_loc}" rpy="0 0 0"/>
       <parent link="${parent}"/>
-      <child link="standoff_209mm_${number}_link"/>
-    </joint>
-    <link name="standoff_209mm_${number}_link">
+      <child link="standoff_251mm_${number}_link"/>
+    </joint>
+    <link name="standoff_251mm_${number}_link">
       <visual>
         <origin xyz=" 0 0 0" rpy="0 0 0"/>
         <geometry>
-          <mesh filename="package://turtlebot_description/meshes/stacks/interbotix/standoff_209mm.stl"/>
+          <mesh filename="package://turtlebot_description/meshes/stacks/interbotix/251mm_Spacer.stl"/>
         </geometry>
         <xacro:insert_block name="material_pink"/>
@@ -137,9 +153,9 @@
         <origin xyz="0 0 0" rpy="0 0 0"/>
         <geometry>
-          <cylinder length="0.209" radius="0.012"/>
-        </geometry>
-      </collision>
-      <inertial>
-        <mass value="0.060"/>
+          <cylinder length="${STANDOFF_251_HEIGHT}" radius="0.012"/>
+        </geometry>
+      </collision>
+      <inertial>
+        <mass value="0.031"/>
         <origin xyz="0 0 0"/>
         <inertia ixx="0.000206991" ixy="0.0" ixz="0.0"
@@ -148,5 +164,5 @@
       </inertial>
     </link>
-    <gazebo reference="standoff_209mm_${number}_link">
+    <gazebo reference="standoff_251mm_${number}_link">
       <material>Gazebo/Black</material>
       <selfCollide>true</selfCollide>
@@ -160,12 +176,12 @@
   -->
   <xacro:macro name="stack_interbotix" params="parent">
-    <standoff_38mm parent="${parent}" number="0" x_loc= "0.120" y_loc= "0.082" z_loc="0.107"/>
-    <standoff_38mm parent="${parent}" number="1" x_loc= "0.055" y_loc= "0.120" z_loc="0.107"/>
-    <standoff_38mm parent="${parent}" number="2" x_loc="-0.055" y_loc= "0.120" z_loc="0.107"/>
-    <standoff_38mm parent="${parent}" number="3" x_loc= "0.120" y_loc="-0.082" z_loc="0.107"/>
-    <standoff_38mm parent="${parent}" number="4" x_loc= "0.055" y_loc="-0.120" z_loc="0.107"/>
-    <standoff_38mm parent="${parent}" number="5" x_loc="-0.055" y_loc="-0.120" z_loc="0.107"/>
+    <standoff_38mm parent="${parent}" number="0" x_loc= "0.120" y_loc= "0.082" z_loc="${STANDOFF_BOTTOM_Z}"/>
+    <standoff_38mm parent="${parent}" number="1" x_loc= "0.055" y_loc= "0.120" z_loc="${STANDOFF_BOTTOM_Z}"/>
+    <standoff_38mm parent="${parent}" number="2" x_loc="-0.055" y_loc= "0.120" z_loc="${STANDOFF_BOTTOM_Z}"/>
+    <standoff_38mm parent="${parent}" number="3" x_loc= "0.120" y_loc="-0.082" z_loc="${STANDOFF_BOTTOM_Z}"/>
+    <standoff_38mm parent="${parent}" number="4" x_loc= "0.055" y_loc="-0.120" z_loc="${STANDOFF_BOTTOM_Z}"/>
+    <standoff_38mm parent="${parent}" number="5" x_loc="-0.055" y_loc="-0.120" z_loc="${STANDOFF_BOTTOM_Z}"/>
     <joint name="plate_bottom_joint" type="fixed">
-      <origin xyz="0.0 0.0 0.1285" rpy="0 0 0"/>
+      <origin xyz="0.0 0.0 ${PLATE_BOTTOM_Z}" rpy="0 0 0"/>
       <parent link="${parent}"/>
       <child link="plate_bottom_link"/>
@@ -175,5 +191,5 @@
         <origin xyz="0 0 0" rpy="0 0 0"/>
         <geometry>
-          <mesh filename="package://turtlebot_description/meshes/stacks/interbotix/plate_bottom.stl"/>
+          <mesh filename="package://turtlebot_description/meshes/stacks/interbotix/TurtleBot2i_BottomPlate.stl"/>
         </geometry>
         <xacro:insert_block name="material_near_black"/>
@@ -186,5 +202,5 @@
       </collision>
       <inertial>
-        <mass value="0.520" />
+        <mass value="0.311" />
         <origin xyz="0 0 0" />
         <inertia ixx="0.003328" ixy="0.0" ixz="0.0"
@@ -198,12 +214,12 @@
       <gravity>true</gravity>
     </gazebo>
-    <standoff_51mm parent="${parent}" number="0" x_loc= "0.069" y_loc= "0.130" z_loc="0.1565"/>
-    <standoff_51mm parent="${parent}" number="1" x_loc= "0.069" y_loc="-0.130" z_loc="0.1565"/>
-    <standoff_51mm parent="${parent}" number="2" x_loc= "-0.001" y_loc= "0.162" z_loc="0.1565"/>
-    <standoff_51mm parent="${parent}" number="3" x_loc= "-0.001" y_loc="-0.162" z_loc="0.1565"/>
-    <standoff_51mm parent="${parent}" number="4" x_loc="-0.104" y_loc= "0.098" z_loc="0.1565"/>
-    <standoff_51mm parent="${parent}" number="5" x_loc="-0.104" y_loc="-0.098" z_loc="0.1565"/>
+    <standoff_51mm parent="${parent}" number="0" x_loc= "0.069" y_loc= "0.130" z_loc="${STANDOFF_MIDDLE_Z}"/>
+    <standoff_51mm parent="${parent}" number="1" x_loc= "0.069" y_loc="-0.130" z_loc="${STANDOFF_MIDDLE_Z}"/>
+    <standoff_51mm parent="${parent}" number="2" x_loc= "-0.001" y_loc= "0.162" z_loc="${STANDOFF_MIDDLE_Z}"/>
+    <standoff_51mm parent="${parent}" number="3" x_loc= "-0.001" y_loc="-0.162" z_loc="${STANDOFF_MIDDLE_Z}"/>
+    <standoff_51mm parent="${parent}" number="4" x_loc="-0.104" y_loc= "0.098" z_loc="${STANDOFF_MIDDLE_Z}"/>
+    <standoff_51mm parent="${parent}" number="5" x_loc="-0.104" y_loc="-0.098" z_loc="${STANDOFF_MIDDLE_Z}"/>
     <joint name="plate_middle_joint" type="fixed">
-      <origin xyz="0.0 0.0 0.1845" rpy="0 0 0"/>
+      <origin xyz="0.0 0.0 ${PLATE_MIDDLE_Z}" rpy="0 0 0"/>
       <parent link="${parent}"/>
       <child link="plate_middle_link"/>
@@ -213,5 +229,5 @@
         <origin xyz="0 0 0" rpy="0 0 0"/>
         <geometry>
-          <mesh filename="package://turtlebot_description/meshes/stacks/interbotix/plate_middle.stl"/>
+          <mesh filename="package://turtlebot_description/meshes/stacks/interbotix/TurtleBot2i_MiddlePlate.stl"/>
         </geometry>
         <xacro:insert_block name="material_near_black"/>
@@ -220,9 +236,9 @@
         <origin xyz="0.0 0.0 0.0" rpy="0 0 0"/>
         <geometry>
-          <mesh filename="package://turtlebot_description/meshes/stacks/interbotix/plate_middle.stl" scale="1.1 1.1 1.1"/>
-        </geometry>
-      </collision>
-      <inertial>
-        <mass value="0.520" />
+          <mesh filename="package://turtlebot_description/meshes/stacks/interbotix/TurtleBot2i_MiddlePlate.stl"/>
+        </geometry>
+      </collision>
+      <inertial>
+        <mass value="0.299" />
         <origin xyz="0 0 0" />
         <inertia ixx="0.003328" ixy="0.0" ixz="0.0"
@@ -236,10 +252,10 @@
       <gravity>true</gravity>
     </gazebo>
-    <standoff_38mm parent="${parent}" number="6" x_loc= "-0.001" y_loc= "0.162" z_loc="0.206"/>
-    <standoff_38mm parent="${parent}" number="7" x_loc= "-0.001" y_loc="-0.162" z_loc="0.206"/>
-    <standoff_38mm parent="${parent}" number="8" x_loc="-0.104" y_loc= "0.098" z_loc="0.206"/>
-    <standoff_38mm parent="${parent}" number="9" x_loc="-0.104" y_loc="-0.098" z_loc="0.206"/>
+    <standoff_81mm parent="${parent}" number="6" x_loc= "-0.001" y_loc= "0.162" z_loc="${STANDOFF_UTILITY_BOTTOM_Z}"/>
+    <standoff_81mm parent="${parent}" number="7" x_loc= "-0.001" y_loc="-0.162" z_loc="${STANDOFF_UTILITY_BOTTOM_Z}"/>
+    <standoff_81mm parent="${parent}" number="8" x_loc="-0.104" y_loc= "0.098" z_loc="${STANDOFF_UTILITY_BOTTOM_Z}"/>
+    <standoff_81mm parent="${parent}" number="9" x_loc="-0.104" y_loc="-0.098" z_loc="${STANDOFF_UTILITY_BOTTOM_Z}"/>
     <joint name="plate_utility_lower" type="fixed">
-      <origin xyz="0.0 0.0 0.2655" rpy="0 0 0"/>
+      <origin xyz="0.0 0.0 ${PLATE_UTILITY_BOTTOM_Z}" rpy="0 0 0"/>
       <parent link="${parent}"/>
       <child link="plate_utility_lower_link"/>
@@ -249,5 +265,5 @@
         <origin xyz="0 0 0" rpy="0 0 0"/>
         <geometry>
-          <mesh filename="package://turtlebot_description/meshes/stacks/interbotix/plate_utility.stl"/>
+          <mesh filename="package://turtlebot_description/meshes/stacks/interbotix/TurtleBot2i_CameraPlate.stl"/>
         </geometry>
         <xacro:insert_block name="material_near_black"/>
@@ -256,9 +272,9 @@
         <origin xyz="0.0 0.0 0.0" rpy="0 0 0"/>
         <geometry>
-          <mesh filename="package://turtlebot_description/meshes/stacks/interbotix/plate_utility.stl"/>
-        </geometry>
-      </collision>
-      <inertial>
-        <mass value="0.520" />
+          <mesh filename="package://turtlebot_description/meshes/stacks/interbotix/TurtleBot2i_CameraPlate.stl"/>
+        </geometry>
+      </collision>
+      <inertial>
+        <mass value="0.151" />
         <origin xyz="0 0 0" />
         <inertia ixx="0.003328" ixy="0.0" ixz="0.0"
@@ -272,10 +288,10 @@
       <gravity>true</gravity>
     </gazebo>
-    <standoff_124mm parent="${parent}" number="0" x_loc= "-0.001" y_loc= "0.162" z_loc="0.292"/>
-    <standoff_124mm parent="${parent}" number="1" x_loc= "-0.001" y_loc="-0.162" z_loc="0.292"/>
-    <standoff_124mm parent="${parent}" number="2" x_loc="-0.104" y_loc= "0.098" z_loc="0.292"/>
-    <standoff_124mm parent="${parent}" number="3" x_loc="-0.104" y_loc="-0.098" z_loc="0.292"/>
+    <standoff_81mm parent="${parent}" number="0" x_loc= "-0.001" y_loc= "0.162" z_loc="${STANDOFF_UTILITY_UPPER_Z}"/>
+    <standoff_81mm parent="${parent}" number="1" x_loc= "-0.001" y_loc="-0.162" z_loc="${STANDOFF_UTILITY_UPPER_Z}"/>
+    <standoff_81mm parent="${parent}" number="2" x_loc="-0.104" y_loc= "0.098" z_loc="${STANDOFF_UTILITY_UPPER_Z}"/>
+    <standoff_81mm parent="${parent}" number="3" x_loc="-0.104" y_loc="-0.098" z_loc="${STANDOFF_UTILITY_UPPER_Z}"/>
     <joint name="plate_utility_upper" type="fixed">
-      <origin xyz="0.0 0.0 0.3565" rpy="0 0 0"/>
+      <origin xyz="0.0 0.0 ${PLATE_UTILITY_UPPER_Z}" rpy="0 0 0"/>
       <parent link="${parent}"/>
       <child link="plate_utility_upper_link"/>
@@ -285,5 +301,5 @@
         <origin xyz="0 0 0" rpy="0 0 0"/>
         <geometry>
-          <mesh filename="package://turtlebot_description/meshes/stacks/interbotix/plate_utility.stl"/>
+          <mesh filename="package://turtlebot_description/meshes/stacks/interbotix/TurtleBot2i_UtilityPlate.stl"/>
         </geometry>
         <xacro:insert_block name="material_near_black"/>
@@ -292,9 +308,9 @@
         <origin xyz="0.0 0.0 0.0" rpy="0 0 0"/>
         <geometry>
-          <mesh filename="package://turtlebot_description/meshes/stacks/interbotix/plate_utility.stl"/>
-        </geometry>
-      </collision>
-      <inertial>
-        <mass value="0.520" />
+          <mesh filename="package://turtlebot_description/meshes/stacks/interbotix/TurtleBot2i_UtilityPlate.stl"/>
+        </geometry>
+      </collision>
+      <inertial>
+        <mass value="0.153" />
         <origin xyz="0 0 0" />
         <inertia ixx="0.003328" ixy="0.0" ixz="0.0"
@@ -308,10 +324,10 @@
       <gravity>true</gravity>
     </gazebo>
-    <standoff_38mm parent="${parent}" number="10" x_loc= "-0.001" y_loc= "0.162" z_loc="0.378"/>
-    <standoff_38mm parent="${parent}" number="11" x_loc= "-0.001" y_loc="-0.162" z_loc="0.378"/>
-    <standoff_38mm parent="${parent}" number="12" x_loc="-0.104" y_loc= "0.098" z_loc="0.378"/>
-    <standoff_38mm parent="${parent}" number="13" x_loc="-0.104" y_loc="-0.098" z_loc="0.378"/>
+    <standoff_81mm parent="${parent}" number="10" x_loc= "-0.001" y_loc= "0.162" z_loc="${STANDOFF_TOP_Z}"/>
+    <standoff_81mm parent="${parent}" number="11" x_loc= "-0.001" y_loc="-0.162" z_loc="${STANDOFF_TOP_Z}"/>
+    <standoff_81mm parent="${parent}" number="12" x_loc="-0.104" y_loc= "0.098" z_loc="${STANDOFF_TOP_Z}"/>
+    <standoff_81mm parent="${parent}" number="13" x_loc="-0.104" y_loc="-0.098" z_loc="${STANDOFF_TOP_Z}"/>
     <joint name="plate_top_joint" type="fixed">
-      <origin xyz="0.0 0.0 0.4375" rpy="0 0 0"/>
+      <origin xyz="0.0 0.0 ${PLATE_TOP_Z}" rpy="0 0 0"/>
       <parent link="${parent}"/>
       <child link="plate_top_link"/>
@@ -321,16 +337,16 @@
         <origin xyz="0 0 0" rpy="0 0 0"/>
         <geometry>
-          <mesh filename="package://turtlebot_description/meshes/stacks/interbotix/plate_top.stl"/>
-        </geometry>
-        <xacro:insert_block name="material_near_black"/>
-      </visual>
-      <collision>
-        <origin xyz="0 0 0" rpy="0 0 0"/>
-        <geometry>
-          <mesh filename="package://turtlebot_description/meshes/stacks/interbotix/plate_top.stl" scale="1.0 1.0 2.0"/>
-        </geometry>
-      </collision>
-      <inertial>
-        <mass value="0.520"/>
+          <mesh filename="package://turtlebot_description/meshes/stacks/interbotix/TurtleBot2i_TopPlate.stl"/>
+        </geometry>
+        <xacro:insert_block name="material_near_black"/>
+      </visual>
+      <collision>
+        <origin xyz="0 0 0" rpy="0 0 0"/>
+        <geometry>
+          <mesh filename="package://turtlebot_description/meshes/stacks/interbotix/TurtleBot2i_TopPlate.stl"/>
+        </geometry>
+      </collision>
+      <inertial>
+        <mass value="0.377"/>
         <origin xyz="0 0 0"/>
         <inertia ixx="0.003328" ixy="0.0" ixz="0.0"
@@ -344,6 +360,6 @@
       <gravity>true</gravity>
     </gazebo>
-    <standoff_209mm parent="${parent}" number="0" x_loc= "0.069" y_loc= "0.130" z_loc="0.292"/>
-    <standoff_209mm parent="${parent}" number="1" x_loc= "0.069" y_loc="-0.130" z_loc="0.292"/>
+    <standoff_251mm parent="${parent}" number="0" x_loc= "0.069" y_loc= "0.130" z_loc="${STANDOFF_FRONT_Z}"/>
+    <standoff_251mm parent="${parent}" number="1" x_loc= "0.069" y_loc="-0.130" z_loc="${STANDOFF_FRONT_Z}"/>
   </xacro:macro>
 </robot>
