Commit message: Restored Astra or ZR300 compatibility

File: turtlebot2i_description/urdf/sensors/astra.urdf.xacro (robot description, xacro)
@@ -6,5 +6,5 @@
   <xacro:property name="astra_cam_px" value="-0.050"/>
   <xacro:property name="astra_cam_py" value="0.0"/>
-  <xacro:property name="astra_cam_pz" value="0.2635"/>
+  <xacro:property name="astra_cam_pz" value="0.3051"/>
   <xacro:property name="astra_depth_rel_rgb_py" value="0.038" />
   <xacro:property name="astra_cam_rel_rgb_py"   value="0.012" />

File: turtlebot2i_description/urdf/sensors/zr300.urdf.xacro (robot description, xacro)
@@ -6,5 +6,5 @@
   <xacro:property name="zr300_origin_x" value="-0.050"/>
   <xacro:property name="zr300_origin_y" value="0.0"/>
-  <xacro:property name="zr300_origin_z" value="0.268"/>
+  <xacro:property name="zr300_origin_z" value="0.2705"/>
   <xacro:property name="zr300_rgb_x" value="0.0"/>
   <xacro:property name="zr300_rgb_y" value="-0.028"/>

Commit message: Astra URDF tidy

File: turtlebot2i_description/urdf/sensors/astra.urdf.xacro (robot description, xacro)
@@ -6,8 +6,7 @@
   <xacro:property name="astra_cam_px" value="-0.050"/>
   <xacro:property name="astra_cam_py" value="0.0"/>
-  <xacro:property name="astra_cam_pz" value="0.3051"/>
+  <xacro:property name="astra_cam_pz" value="0.3051"/> <!--Sensor base is ~34.6mm below origin-->
   <xacro:property name="astra_depth_rel_rgb_py" value="0.038" />
   <xacro:property name="astra_cam_rel_rgb_py"   value="0.012" />
-  <xacro:property name="astra_dae_display_scale"   value="1.0" />
   <!-- Parameterised in part by properties above -->
   <xacro:macro name="sensor_astra" params="parent">
@@ -35,5 +34,5 @@
         <origin xyz="0 0 0" rpy="0 0 0"/>
         <geometry>
-          <mesh filename="package://turtlebot2i_description/meshes/sensors/astra_new.stl" scale="${astra_dae_display_scale} ${astra_dae_display_scale} ${astra_dae_display_scale}"/>
+          <mesh filename="package://turtlebot2i_description/meshes/sensors/astra_new.stl"/>
         </geometry>
         <xacro:insert_block name="material_black"/>

Commit message: Refactoring to camera_navigation and camera_floor

File: turtlebot2i_description/urdf/sensors/astra.urdf.xacro (robot description, xacro)
@@ -11,24 +11,24 @@
   <!-- Parameterised in part by properties above -->
   <xacro:macro name="sensor_astra" params="parent">
-    <joint name="camera_rgb_joint" type="fixed">
+    <joint name="camera_navigation_rgb_joint" type="fixed">
       <origin xyz="${astra_cam_px} ${astra_cam_py} ${astra_cam_pz}"
               rpy="0 0 0"/>
       <parent link="${parent}"/>
-      <child link="camera_rgb_frame" />
+      <child link="camera_navigation_rgb_frame" />
     </joint>
-    <link name="camera_rgb_frame"/>
-    <joint name="camera_rgb_optical_joint" type="fixed">
+    <link name="camera_navigation_rgb_frame"/>
+    <joint name="camera_navigation_rgb_optical_joint" type="fixed">
       <origin xyz="0 ${astra_cam_rel_rgb_py} 0" rpy="${-M_PI/2} 0 ${-M_PI/2}" />
-      <parent link="camera_rgb_frame" />
-      <child link="camera_rgb_optical_frame" />
+      <parent link="camera_navigation_rgb_frame" />
+      <child link="camera_navigation_rgb_optical_frame" />
     </joint>
-    <link name="camera_rgb_optical_frame"/>
-    <joint name="camera_joint" type="fixed">
+    <link name="camera_navigation_rgb_optical_frame"/>
+    <joint name="camera_navigation_joint" type="fixed">
       <origin xyz="0 0 0"
               rpy="0 0 0"/>
-      <parent link="camera_rgb_frame"/>
-      <child link="camera_link"/>
+      <parent link="camera_navigation_rgb_frame"/>
+      <child link="camera_navigation_link"/>
     </joint>
-    <link name="camera_link">
+    <link name="camera_navigation_link">
       <visual>
         <origin xyz="0 0 0" rpy="0 0 0"/>
@@ -52,21 +52,21 @@
       </inertial>
     </link>
-    <gazebo reference="camera_link">
+    <gazebo reference="camera_navigation_link">
       <material>Gazebo/Blue</material>
       <selfCollide>true</selfCollide>
       <gravity>true</gravity>
     </gazebo>
-    <joint name="camera_depth_joint" type="fixed">
+    <joint name="camera_navigation_depth_joint" type="fixed">
       <origin xyz="0 ${astra_depth_rel_rgb_py} 0" rpy="0 0 0" />
-      <parent link="camera_rgb_frame" />
-      <child link="camera_depth_frame" />
+      <parent link="camera_navigation_rgb_frame" />
+      <child link="camera_navigation_depth_frame" />
     </joint>
-    <link name="camera_depth_frame"/>
-    <joint name="camera_depth_optical_joint" type="fixed">
+    <link name="camera_navigation_depth_frame"/>
+    <joint name="camera_navigation_depth_optical_joint" type="fixed">
       <origin xyz="0 0 0" rpy="${-M_PI/2} 0 ${-M_PI/2}" />
-      <parent link="camera_depth_frame" />
-      <child link="camera_depth_optical_frame" />
+      <parent link="camera_navigation_depth_frame" />
+      <child link="camera_navigation_depth_optical_frame" />
     </joint>
-    <link name="camera_depth_optical_frame"/>
+    <link name="camera_navigation_depth_optical_frame"/>
     <!-- RGBD sensor for simulation, same as Kinect -->
     <turtlebot_sim_3dsensor/>

File: turtlebot2i_description/urdf/sensors/sr300.urdf.xacro (robot description, xacro)
@@ -21,11 +21,11 @@
     ==  Intel SR300 body joints & links ==
     -->
-    <!-- camera_sr300 body -->
-    <joint name="camera_sr300_joint" type="fixed">
+    <!-- camera_floor body -->
+    <joint name="camera_floor_joint" type="fixed">
       <origin xyz="${sr300_cam_offset_px} ${sr300_cam_offset_py} ${sr300_cam_offset_pz}" rpy="0 1.16 0"/>
       <parent link="${parent}"/>
-      <child link="camera_sr300" />
+      <child link="camera_floor" />
     </joint>
-    <link name="camera_sr300">
+    <link name="camera_floor">
       <visual>
        <origin xyz="0 0 0" rpy="0 0 0"/>
@@ -50,5 +50,5 @@
       </inertial>
     </link>
-    <gazebo reference="camera_sr300">
+    <gazebo reference="camera_floor">
       <material>Gazebo/Blue</material>
       <selfCollide>true</selfCollide>
@@ -58,34 +58,34 @@
     ==  RGB joints & links ==
     -->
-    <joint name="camera_sr300_rgb_joint" type="fixed">
+    <joint name="camera_floor_rgb_joint" type="fixed">
       <origin xyz="${sr300_cam_rgb_px} ${sr300_cam_rgb_py} ${sr300_cam_rgb_pz}" rpy="0 0 0"/>
-      <parent link="camera_sr300"/>
-      <child link="camera_sr300_rgb_frame" />
+      <parent link="camera_floor"/>
+      <child link="camera_floor_rgb_frame" />
     </joint>
-    <link name="camera_sr300_rgb_frame"/>
-    <joint name="camera_sr300_rgb_optical_joint" type="fixed">
+    <link name="camera_floor_rgb_frame"/>
+    <joint name="camera_floor_rgb_optical_joint" type="fixed">
       <origin xyz="0 0 0" rpy="${-M_PI/2} 0 ${-M_PI/2}" />
-      <parent link="camera_sr300_rgb_frame" />
-      <child link="camera_sr300_rgb_optical_frame" />
+      <parent link="camera_floor_rgb_frame" />
+      <child link="camera_floor_rgb_optical_frame" />
     </joint>
-    <link name="camera_sr300_rgb_optical_frame"/>
+    <link name="camera_floor_rgb_optical_frame"/>
     <!--
     ==  Depth joints & links ==
     -->
-    <joint name="camera_sr300_depth_joint" type="fixed">
+    <joint name="camera_floor_depth_joint" type="fixed">
         <origin xyz="0 ${sr300_cam_depth_offset} 0" rpy="0 0 0" />
-        <parent link="camera_sr300_rgb_frame" />
-        <child link="camera_sr300_depth_frame" />
+        <parent link="camera_floor_rgb_frame" />
+        <child link="camera_floor_depth_frame" />
     </joint>
-    <link name="camera_sr300_depth_frame"/>
-    <joint name="camera_sr300_depth_optical_joint" type="fixed">
+    <link name="camera_floor_depth_frame"/>
+    <joint name="camera_floor_depth_optical_joint" type="fixed">
         <origin xyz="0 0 0" rpy="${-M_PI/2} 0 ${-M_PI/2}" />
-        <parent link="camera_sr300_depth_frame" />
-        <child link="camera_sr300_depth_optical_frame" />
+        <parent link="camera_floor_depth_frame" />
+        <child link="camera_floor_depth_optical_frame" />
     </joint>
-    <link name="camera_sr300_depth_optical_frame"/>
+    <link name="camera_floor_depth_optical_frame"/>
   	<!-- Simulation sensor -->
-    <gazebo reference="camera_sr300">
-      <sensor type="depth" name="camera_sr300">
+    <gazebo reference="camera_floor">
+      <sensor type="depth" name="camera_floor">
         <always_on>true</always_on>
         <update_rate>20.0</update_rate>
@@ -103,5 +103,5 @@
         </camera>
         <plugin name="kinect_camera_controller" filename="libgazebo_ros_openni_kinect.so">
-          <cameraName>camera_sr300</cameraName>
+          <cameraName>camera_floor</cameraName>
           <alwaysOn>true</alwaysOn>
           <updateRate>10</updateRate>
@@ -111,5 +111,5 @@
           <cameraInfoTopicName>rgb/camera_info</cameraInfoTopicName>
           <depthImageCameraInfoTopicName>depth/camera_info</depthImageCameraInfoTopicName>
-          <frameName>camera_sr300_depth_optical_frame</frameName>
+          <frameName>camera_floor_depth_optical_frame</frameName>
           <baseline>0.1</baseline>
           <distortion_k1>0.0</distortion_k1>

File: turtlebot2i_description/urdf/sensors/zr300.urdf.xacro (robot description, xacro)
@@ -14,11 +14,11 @@
   <xacro:macro name="sensor_zr300" params="parent">
     <!--Sensor body-->
-    <joint name="camera_joint" type="fixed">
+    <joint name="camera_navigation_joint" type="fixed">
       <origin xyz="${zr300_origin_x} ${zr300_origin_y} ${zr300_origin_z}"
               rpy="0 0 0"/>
       <parent link="${parent}"/>
-      <child link="camera_link"/>
+      <child link="camera_navigation_link"/>
     </joint>
-    <link name="camera_link">
+    <link name="camera_navigation_link">
       <visual>
         <origin xyz="0 0 0" rpy="0 0 0"/>
@@ -43,5 +43,5 @@
       </inertial>
     </link>
-    <gazebo reference="camera_link">
+    <gazebo reference="camera_navigation_link">
       <material>Gazebo/Blue</material>
       <selfCollide>true</selfCollide>
@@ -49,42 +49,42 @@
     </gazebo>
     <!--RGB-->
-    <joint name="camera_rgb_joint" type="fixed">
+    <joint name="camera_navigation_rgb_joint" type="fixed">
       <origin xyz="${zr300_rgb_x} ${zr300_rgb_y} ${zr300_rgb_z}" rpy="0 0 0"/>
-      <parent link="camera_link"/>
-      <child link="camera_rgb_frame" />
+      <parent link="camera_navigation_link"/>
+      <child link="camera_navigation_rgb_frame" />
     </joint>
-    <link name="camera_rgb_frame"/>
-    <joint name="camera_rgb_optical_joint" type="fixed">
+    <link name="camera_navigation_rgb_frame"/>
+    <joint name="camera_navigation_rgb_optical_joint" type="fixed">
       <origin xyz="0 0 0" rpy="${-M_PI/2} 0 ${-M_PI/2}" />
-      <parent link="camera_rgb_frame" />
-      <child link="camera_rgb_optical_frame" />
+      <parent link="camera_navigation_rgb_frame" />
+      <child link="camera_navigation_rgb_optical_frame" />
     </joint>
-    <link name="camera_rgb_optical_frame"/>
+    <link name="camera_navigation_rgb_optical_frame"/>
     <!--Depth-->
-    <joint name="camera_depth_joint" type="fixed">
+    <joint name="camera_navigation_depth_joint" type="fixed">
       <origin xyz="0 ${zr300_depth_y} 0" rpy="0 0 0" />
-      <parent link="camera_rgb_frame" />
-      <child link="camera_depth_frame" />
+      <parent link="camera_navigation_rgb_frame" />
+      <child link="camera_navigation_depth_frame" />
     </joint>
-    <link name="camera_depth_frame"/>
-    <joint name="camera_depth_optical_joint" type="fixed">
+    <link name="camera_navigation_depth_frame"/>
+    <joint name="camera_navigation_depth_optical_joint" type="fixed">
       <origin xyz="0 0 0" rpy="${-M_PI/2} 0 ${-M_PI/2}" />
-      <parent link="camera_depth_frame" />
-      <child link="camera_depth_optical_frame" />
+      <parent link="camera_navigation_depth_frame" />
+      <child link="camera_navigation_depth_optical_frame" />
     </joint>
-    <link name="camera_depth_optical_frame"/>
+    <link name="camera_navigation_depth_optical_frame"/>
     <!--FishEye-->
-    <joint name="camera_fisheye_joint" type="fixed">
+    <joint name="camera_navigation_fisheye_joint" type="fixed">
       <origin xyz="0 ${zr300_fisheye_y} 0" rpy="0 0 0" />
-      <parent link="camera_rgb_frame" />
-      <child link="camera_fisheye_frame" />
+      <parent link="camera_navigation_rgb_frame" />
+      <child link="camera_navigation_fisheye_frame" />
     </joint>
-    <link name="camera_fisheye_frame"/>
-    <joint name="camera_fisheye_optical_joint" type="fixed">
+    <link name="camera_navigation_fisheye_frame"/>
+    <joint name="camera_navigation_fisheye_optical_joint" type="fixed">
       <origin xyz="0 0 0" rpy="${-M_PI/2} 0 ${-M_PI/2}" />
-      <parent link="camera_fisheye_frame" />
-      <child link="camera_fisheye_optical_frame" />
+      <parent link="camera_navigation_fisheye_frame" />
+      <child link="camera_navigation_fisheye_optical_frame" />
     </joint>
-    <link name="camera_fisheye_optical_frame"/>
+    <link name="camera_navigation_fisheye_optical_frame"/>
     <!-- RGBD sensor for simulation, same as Kinect -->
     <turtlebot_sim_3dsensor/>
