Commit message: Adjusted ZR300, just in case.

File: turtlebot2i_description/urdf/sensors/zr300.urdf.xacro (robot description, xacro)
@@ -6,5 +6,5 @@
   <xacro:property name="zr300_origin_x" value="-0.050"/>
   <xacro:property name="zr300_origin_y" value="0.0"/>
-  <xacro:property name="zr300_origin_z" value="0.2705"/>
+  <xacro:property name="zr300_origin_z" value="0.25"/>
   <xacro:property name="zr300_rgb_x" value="0.0"/>
   <xacro:property name="zr300_rgb_y" value="-0.028"/>
