Commit message: Updates as of 6/14/2020:
 1) Replaces the outdated realsense-camera and librealsense packages with the updated realsense2_camera and librealsense2 packages. This will be outlined in the full build instructions shortly.
 2) No need for the kobuki udev rule since the kobuki_node does this automatically. Similarly, no need to look up the serial number for the arbotix - the rule is now that any ftdi cable that is not for a kobuki is defined as 'arbotix'

File: turtlebot2i_description/urdf/sensors/sr300.urdf.xacro (robot description, xacro)
@@ -52,16 +52,16 @@
     ==  RGB joints & links ==
     -->
-    <joint name="camera_sr300_rgb_joint" type="fixed">
+    <joint name="camera_sr300_color_joint" type="fixed">
       <origin xyz="${sr300_cam_rgb_px} ${sr300_cam_rgb_py} ${sr300_cam_rgb_pz}" rpy="0 1.16 0"/>
       <parent link="camera_sr300"/>
-      <child link="camera_sr300_rgb_frame" />
+      <child link="camera_sr300_color_frame" />
     </joint>
-    <link name="camera_sr300_rgb_frame"/>
-    <joint name="camera_sr300_rgb_optical_joint" type="fixed">
+    <link name="camera_sr300_color_frame"/>
+    <joint name="camera_sr300_color_optical_joint" type="fixed">
       <origin xyz="0 0 0" rpy="${-M_PI/2} 0 ${-M_PI/2}" />
-      <parent link="camera_sr300_rgb_frame" />
-      <child link="camera_sr300_rgb_optical_frame" />
+      <parent link="camera_sr300_color_frame" />
+      <child link="camera_sr300_color_optical_frame" />
     </joint>
-    <link name="camera_sr300_rgb_optical_frame"/>
+    <link name="camera_sr300_color_optical_frame"/>
     <!--
     ==  Depth joints & links ==
@@ -69,5 +69,5 @@
     <joint name="camera_sr300_depth_joint" type="fixed">
         <origin xyz="0 ${sr300_cam_depth_offset} 0" rpy="0 0 0" />
-        <parent link="camera_sr300_rgb_frame" />
+        <parent link="camera_sr300_color_frame" />
         <child link="camera_sr300_depth_frame" />
     </joint>
