Commit message: Updates as of 6/24/2020:
 1) Added launch file to just launch the Turtlebot2i robot description in Rviz (no robot necessary)
 2) Modified the top plate and SR300 camera STLS with the new SR305 camera.
 3) Modified the SR300 URDF to make the camera frame placement correct
 4) Parent of SR300 sensor is now 'plate_top_link' instead of 'base_link'.

File: turtlebot2i_description/robots/kobuki_interbotix_astra.urdf.xacro (robot description, xacro)
@@ -11,5 +11,5 @@
   <stack_interbotix parent="base_link"/>
   <sensor_astra parent="base_link"/>
-  <sensor_sr300 parent="base_link"/>
+  <sensor_sr300 parent="plate_top_link"/>
   <phantomx_pincher_arm parent="base_link" color="Red" gripper_color="Red">
     <origin xyz="0.145 0.0 0.124"/>

File: turtlebot2i_description/urdf/sensors/sr300.urdf.xacro (robot description, xacro)
@@ -4,11 +4,10 @@
   <xacro:include filename="$(find turtlebot2i_description)/urdf/turtlebot_properties.urdf.xacro"/>
   <!-- Intel SR300 parameters -->
-  <xacro:property name="sr300_cam_offset_px" value="0.138" />
+  <xacro:property name="sr300_cam_offset_px" value="0.120" />
   <xacro:property name="sr300_cam_offset_py" value="0.0" />
-  <xacro:property name="sr300_cam_offset_pz" value="0.444" />
+  <xacro:property name="sr300_cam_offset_pz" value="0.0023" />
   <xacro:property name="sr300_cam_rgb_px" value="0.0"/>
-  <xacro:property name="sr300_cam_rgb_py" value="0.003"/>
+  <xacro:property name="sr300_cam_rgb_py" value="0.02403"/>
   <xacro:property name="sr300_cam_rgb_pz" value="0.0"/>
-  <xacro:property name="sr300_cam_depth_offset" value="-0.024"/>
   <xacro:macro name="sensor_sr300" params="parent">
     <!--
@@ -16,21 +15,21 @@
     -->
     <!-- camera_sr300 body -->
-    <joint name="camera_sr300_joint" type="fixed">
+    <joint name="camera_sr300_assembly_joint" type="fixed">
       <origin xyz="${sr300_cam_offset_px} ${sr300_cam_offset_py} ${sr300_cam_offset_pz}" rpy="0 0 0"/>
       <parent link="${parent}"/>
-      <child link="camera_sr300" />
+      <child link="camera_sr300_assembly"/>
     </joint>
-    <link name="camera_sr300">
+    <link name="camera_sr300_assembly">
       <visual>
        <origin xyz="0 0 0" rpy="0 0 0"/>
         <geometry>
-         <mesh filename="package://turtlebot2i_description/meshes/sensors/sr300_tb2i.stl" />
+         <mesh filename="package://turtlebot2i_description/meshes/sensors/sr300_tb2i.stl" scale="0.001 0.001 0.001"/>
         </geometry>
-        <xacro:insert_block name="material_black"/>
+        <xacro:insert_block name="material_grey"/>
       </visual>
       <collision>
         <origin xyz="0.0 0.0 0.0" rpy="0 0 0"/>
         <geometry>
-          <mesh filename="package://turtlebot2i_description/meshes/sensors/sr300_tb2i.stl" scale="2.0 2.0 2.0" />
+          <mesh filename="package://turtlebot2i_description/meshes/sensors/sr300_tb2i.stl" scale="0.001 0.001 0.001"/>
         </geometry>
       </collision>
@@ -44,14 +43,20 @@
       </inertial>
     </link>
-    <gazebo reference="camera_sr300">
+    <gazebo reference="camera_sr300_assembly">
       <material>Gazebo/Blue</material>
       <selfCollide>true</selfCollide>
       <gravity>true</gravity>
     </gazebo>
+    <joint name="camera_sr300_joint" type="fixed">
+      <origin xyz="0.033584 -0.00754 -0.004849" rpy="0 1.15192 0"/>
+      <parent link="camera_sr300_assembly"/>
+      <child link="camera_sr300"/>
+    </joint>
+    <link name="camera_sr300"/>
     <!--
     ==  RGB joints & links ==
     -->
     <joint name="camera_sr300_color_joint" type="fixed">
-      <origin xyz="${sr300_cam_rgb_px} ${sr300_cam_rgb_py} ${sr300_cam_rgb_pz}" rpy="0 1.16 0"/>
+      <origin xyz="${sr300_cam_rgb_px} ${sr300_cam_rgb_py} ${sr300_cam_rgb_pz}" rpy="0 0 0"/>
       <parent link="camera_sr300"/>
       <child link="camera_sr300_color_frame" />
@@ -68,6 +73,6 @@
     -->
     <joint name="camera_sr300_depth_joint" type="fixed">
-        <origin xyz="0 ${sr300_cam_depth_offset} 0" rpy="0 0 0" />
-        <parent link="camera_sr300_color_frame" />
+        <origin xyz="0 0 0" rpy="0 0 0" />
+        <parent link="camera_sr300" />
         <child link="camera_sr300_depth_frame" />
     </joint>

File: turtlebot2i_description/urdf/stacks/interbotix.urdf.xacro (robot description, xacro)
@@ -302,12 +302,12 @@
         <origin xyz="0 0 0" rpy="0 0 0"/>
         <geometry>
-          <mesh filename="package://turtlebot2i_description/meshes/stacks/interbotix/TurtleBot2i_TopPlate.stl"/>
-        </geometry>
-        <xacro:insert_block name="material_near_black"/>
-      </visual>
-      <collision>
-        <origin xyz="0 0 0" rpy="0 0 0"/>
-        <geometry>
-          <mesh filename="package://turtlebot2i_description/meshes/stacks/interbotix/TurtleBot2i_TopPlate.stl"/>
+          <mesh filename="package://turtlebot2i_description/meshes/stacks/interbotix/TurtleBot2i_TopPlate.stl" scale="0.001 0.001 0.001"/>
+        </geometry>
+        <xacro:insert_block name="material_near_black"/>
+      </visual>
+      <collision>
+        <origin xyz="0 0 0" rpy="0 0 0"/>
+        <geometry>
+          <mesh filename="package://turtlebot2i_description/meshes/stacks/interbotix/TurtleBot2i_TopPlate.stl" scale="0.001 0.001 0.001"/>
         </geometry>
       </collision>
